Commit message: add camera

File: urdf/camera.xacro (robot description, xacro)
@@ -4,5 +4,5 @@
         <parent link="chassis"/>
         <child link="camera_link"/>
-        <origin xyz="0.276 0 0.181" rpy="0 0.18 0"/>
+        <origin xyz="0.40 0 0.08" rpy="0 0 0"/>
     </joint>
     <link name="camera_link">

File: urdf/robot.urdf.xacro (robot description, xacro)
@@ -11,5 +11,5 @@
     </xacro:unless>
     <xacro:include filename="lidar.xacro" />
-    <!-- <xacro:include filename="camera.xacro" /> -->
+    <xacro:include filename="camera.xacro" />
     <!-- <xacro:include filename="depth_camera.xacro" /> -->
 </robot>
